File: kicad/stm32card/_autosave-stm32card.kicad_sch (KiCad schematic)
At the start: 83 parts, among them J1 USB_C_Receptacle_PowerOnly_6P, Q1 AO3400A, Q2 AO3400A, Q3 AO3400A, Q4 AO3401A, U1 CN3600, U2 LM66100DCK, U3 LM66100DCK, U4 STM32F103C8T6, U5 N096-1608TBBIG11-H13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

Commit message: pre-readme
Other:
- note removed: "I finished this in a rush and I'm not sure why I did this. R21 should be a short and there needs to be a resistor instead of a diode."
Changed lines of the file:
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@@
-		)
-	)
-	(text "I finished this in a rush and I'm not sure why I did this.\nR21 should be a short and there needs to be a resistor instead of a diode."
-		(exclude_from_sim no)
-		(at 84.074 149.352 0)
-		(effects
-			(font
-				(size 1.27 1.27)
-			)
 		)
 	)
