File: kicad/stm32card/stm32card.kicad_pcb (KiCad board)
At the start: 2 copper layers, 88.9 x 50.8 mm, 82 parts, among them J1 USB_C_Receptacle_PowerOnly_6P, Q1 XR2N13, Q2 XR2N13, U1 CN3600, U2 LM66100DCK, U3 LM66100DCK, U4 STM32F103C8T6, U5 N096-1608TBBIG11-H13, U6 TLV61220DBVR-TP, U7 BU4210G-TR, U9 CJ6300BM

Commit message: quick update for garmin
Parts:
- removed TP1: tp_battery, TestPoint:TestPoint_Pad_D2.0mm
- removed TP_mosi1, TP_sck1: TestPoint, TestPoint:TestPoint_Pad_D2.0mm
- added D4: D_Schottky, Diode_SMD:D_SMA, F.Cu at (150.3, 115.4)
- added D5: 1N4148, Diode_SMD:D_SOD-323, F.Cu at (156.4, 119.6)
- added Q3: AO3400A, Package_TO_SOT_SMD:SOT-23, F.Cu at (159.3, 98.3)
- added Q4: AO3401A, Package_TO_SOT_SMD:SOT-23, F.Cu at (159.3, 94.8)
- added R25: 10k, Resistor_SMD:R_0603_1608Metric, F.Cu at (163.0, 97.4)
- added R26: 1k, Resistor_SMD:R_0603_1608Metric, F.Cu at (166.5, 116.3)
- added R3: 1k, Resistor_SMD:R_0603_1608Metric, F.Cu at (155.8, 97.5)
- BT1: footprint Battery:BatteryHolder_Keystone_2466_1xAAA -> indigos_imports:BAT-SMD_BH-AAA-B5BA021
- C10: value 15nF -> 1uF
- Q1, Q2: value XR2N13 -> AO3400A
- R14, R15: value 50 -> 1k
- R21, R4: value 0 -> 10k
- R22: value 10k -> 0
- R23: value 10k -> 1k
- b_a1, b_b1, b_down1, b_left1, b_right1, b_up1: footprint easyeda2kicad:SW-SMD_4P-L6.0-W6.0-P4.50-LS8.6 -> indigos_imports:SW-SMD_4P-L6.0-W6.0-P4.50-LS8.6
- moved TestPoint_gnd1 52.6 mm to (218.2, 94.9)
- moved R22 39.5 mm to (159.9, 86.6), turned to 0 degrees
- moved R21 38.0 mm to (160.2, 127.1), turned to 180 degrees
- moved R4 27.1 mm to (159.0, 118.7), turned to 0 degrees
- moved D3 18.8 mm to (144.5, 90.8), turned to 90 degrees
- moved BT1 17.3 mm to (189.0, 90.1)
- moved D2 17.0 mm to (146.3, 91.0), turned to 90 degrees
- moved R15 16.6 mm to (146.6, 97.6), turned to 0 degrees
- moved R14 15.0 mm to (148.3, 94.4), turned to -90 degrees
- moved D1 5.52 mm to (157.9, 84.0), turned to 180 degrees
- moved L1 4.97 mm to (151.0, 86.2), turned to 90 degrees
- moved C9 4.73 mm to (148.3, 91.1), turned to -90 degrees
- moved TP2 4.41 mm to (138.3, 91.1)
- moved U1 3.88 mm to (153.6, 93.0)
- moved R23 3.19 mm to (157.6, 124.8), turned to -90 degrees
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Connections:
- net Net-(U2-VIN) renamed bat_3v
- C1 pad 1: Net-(D1-K) -> bat output
- J1 pad SH1: (no net) -> GND
- J1 pad SH2: (no net) -> GND
- J1 pad SH3: (no net) -> GND
- J1 pad SH4: (no net) -> GND
- Q1 pad 1: backlight_fet -> Net-(Q1-G)
- Q1 pad 2: Net-(Q1-S) -> GND
- Q1 pad 3: +3V0 -> Net-(Q1-D)
- Q2 pad 1: usb vbus -> Net-(Q2-G)
- Q2 pad 2: GND -> Net-(Q2-S)
- Q2 pad 3: Net-(Q2-D) -> Net-(D5-K)
- R21 pad 1: Net-(D1-K) -> Net-(Q2-S)
- R21 pad 2: bat output -> GND
- R22 pad 1: usb vbus -> Net-(D1-K)
- R22 pad 2: GND -> bat output
- R23 pad 2: Net-(Q2-D) -> Net-(Q2-G)
- R4 pad 1: Net-(U1-ISEL) -> usb vbus
- U1 pad 2: Net-(U1-ISEL) -> GND
- U3 pad 3: Net-(Q2-D) -> Net-(D5-K)
- U5 pad 11: GND -> Net-(Q1-D)
- U5 pad 12: Net-(Q1-S) -> +3V0
- U9 pad 1: usb vbus -> Net-(D4-K)
- U9 pad 3: usb vbus -> Net-(D4-K)
- b_b1 pad 4: in_button_b -> unconnected-(b_b1-Pad4)
Routing:
- net GND: track 75.7 -> 103.4 mm, vias 41 -> 39
- net usb vbus: track 109.1 -> 84.8 mm
- net Net-(Q1-D): track 0.00 -> 18.7 mm
- net Net-(Q1-S): track 17.5 -> 0.00 mm
- net bat output: track 38.7 -> 54.2 mm
- net Net-(D5-K): track 0.00 -> 10.2 mm
- net Net-(D4-K): track 0.00 -> 8.41 mm
- net Net-(Q2-D): track 7.54 -> 0.00 mm
- net in_button_b: track 30.9 -> 23.8 mm
- net Net-(U1-~{CHRG}): track 3.45 -> 10.4 mm
- net Net-(U1-~{DONE}): track 9.71 -> 3.03 mm
- net Net-(U1-ISEL): track 6.15 -> 0.00 mm
- net Net-(D3-K): track 1.64 -> 6.55 mm
- net bat_3v: track 11.7 -> 16.6 mm
- net Net-(Q3-D): track 0.00 -> 4.85 mm
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Other:
- board text added: "BEFORE RE-ORDERING: - SPI speed stuck at 2mHZ - differential routing? - don't forget stencil!!!! - check 3d model (WITH CORRECT LAYERS AAAAAAAA)"
- board text added: "hold any button to return home"
- board text added: "rechargable AAA NiMH only"
- board text removed: "BEFORE RE-ORDERING: - fix routing to MCU; footprint was changed - fix vtext - SPI NSI - LEDs? - change your god damn test pins - remove if no more needed - remove button outlines - SPI speed stuck at 2mHZ - differential routing? - LCD backlight MOSFTER - test to see if sleep mode is accurate to datasheet - screen responds in sleep mode, which is sus - add mosfet to LED VDD if above is too sus"
